File: TSAL/PCB.kicad_pcb (KiCad board)
At the start: 4 copper layers, 100 x 60 mm, 80 parts, among them J1 TE 770966-2, J2 JST B04B-XASK, J3 Conn_01x02, J4 Conn_01x02, Q1 IRLZ44N, Q2 MMBT3904, Q3 IRLZ44N, U1 TL431D, U2 LMV331, U3 UCC12040DVE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

Commit message: JP1 Edit
Parts:
- JP1: value SolderJumper_2_Bridged -> SolderJumper_2_Open; footprint Jumper:SolderJumper-2_P1.3mm_Bridged_RoundedPad1.0x1.5mm -> Jumper:SolderJumper-2_P1.3mm_Open_RoundedPad1.0x1.5mm
- U6: value LF50_TO252 -> L7805
- moved JP1 0.21 mm to (134.7, 91.2)
Changed lines of the file:
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@@
     )
   )
-  (footprint "Jumper:SolderJumper-2_P1.3mm_Bridged_RoundedPad1.0x1.5mm" (layer "F.Cu")
-    (at 134.6 91)
-    (descr "SMD Solder Jumper, 1x1.5mm, rounded Pads, 0.3mm gap, bridged with 1 copper strip")
-    (tags "net tie solder jumper bridged")
-    (property "Sheetfile" "PCB.kicad_sch")
-    (property "Sheetname" "")
-    (property "ki_description" "Solder Jumper, 2-pole, closed/bridged")
-    (property "ki_keywords" "solder jumper SPST")
-    (attr exclude_from_pos_files)
-    (net_tie_pad_groups "1, 2")
-    (fp_text reference "JP1" (at -2.6 0 90) (layer "F.SilkS")
-        (effects (font (size 1 1) (thickness 0.15)))
-    )
-    (fp_text value "SolderJumper_2_Bridged" (at 0 1.9) (layer "F.Fab")
-        (effects (font (size 1 1) (thickness 0.15)))
-    )
-    (fp_poly
-      (pts
-        (xy 0.25 -0.3)
-        (xy -0.25 -0.3)
-        (xy -0.25 0.3)
-        (xy 0.25 0.3)
-      )
-      (stroke (width 0) (type solid)) (fill solid) (layer "F.Cu"))
-    (fp_line (start -1.4 0.3) (end -1.4 -0.3)
-      (stroke (width 0.12) (type solid)) (layer "F.SilkS"))
-    (fp_line (start -0.7 -1) (end 0.7 -1)
-      (stroke (width 0.12) (type solid)) (layer "F.SilkS"))
-    (fp_line (start 0.7 1) (end -0.7 1)
-      (stroke (width 0.12) (type solid)) (layer "F.SilkS"))
-    (fp_line (start 1.4 -0.3) (end 1.4 0.3)
-      (stroke (width 0.12) (type solid)) (layer "F.SilkS"))
-    (fp_arc (start -1.4 -0.3) (mid -1.194975 -0.794975) (end -0.7 -1)
-      (stroke (width 0.12) (type solid)) (layer "F.SilkS"))
-    (fp_arc (start -0.7 1) (mid -1.194975 0.794975) (end -1.4 0.3)
-      (stroke (width 0.12) (type solid)) (layer "F.SilkS"))
-    (fp_arc (start 0.7 -1) (mid 1.194975 -0.794975) (end 1.4 -0.3)
-      (stroke (width 0.12) (type solid)) (layer "F.SilkS"))
-    (fp_arc (start 1.4 0.3) (mid 1.194975 0.794975) (end 0.7 1)
-      (stroke (width 0.12) (type solid)) (layer "F.SilkS"))
-    (fp_line (start -1.65 -1.25) (end -1.65 1.25)
-      (stroke (width 0.05) (type solid)) (layer "F.CrtYd"))
-    (fp_line (start -1.65 -1.25) (end 1.65 -1.25)
-      (stroke (width 0.05) (type solid)) (layer "F.CrtYd"))
-    (fp_line (start 1.65 1.25) (end -1.65 1.25)
-      (stroke (width 0.05) (type solid)) (layer "F.CrtYd"))
-    (fp_line (start 1.65 1.25) (end 1.65 -1.25)
-      (stroke (width 0.05) (type solid)) (layer "F.CrtYd"))
-    (pad "1" smd custom (at -0.65 0) (size 1 0.5) (layers "F.Cu" "F.Mask")
-      (net 43 "Net-(D6-A)") (pinfunction "A") (pintype "passive") (zone_connect 2)
-      (options (clearance outline) (anchor rect))
-      (primitives
-        (gr_circle (center 0 0.25) (end 0.5 0.25) (width 0) (fill yes))
-        (gr_circle (center 0 -0.25) (end 0.5 -0.25) (width 0) (fill yes))
-        (gr_poly
-          (pts
-            (xy 0.5 0.75)
-            (xy 0 0.75)
-            (xy 0 -0.75)
-            (xy 0.5 -0.75)
-          )
-          (width 0) (fill yes))
-      ))
-    (pad "2" smd custom (at 0.65 0) (size 1 0.5) (layers "F.Cu" "F.Mask")
-      (net 2 "+5V") (pinfunction "B") (pintype "passive") (zone_connect 2)
-      (options (clearance outline) (anchor rect))
-      (primitives
-        (gr_circle (center 0 0.25) (end 0.5 0.25) (width 0) (fill yes))
-        (gr_circle (center 0 -0.25) (end 0.5 -0.25) (width 0) (fill yes))
-        (gr_poly
-          (pts
-            (xy 0 0.75)
-            (xy -0.5 0.75)
-            (xy -0.5 -0.75)
-            (xy 0 -0.75)
-          )
-          (width 0) (fill yes))
-      ))
-  )
   (footprint "TestPoint:TestPoint_Keystone_5019_Minature" (layer "F.Cu")
     (at 134.75 94.5 180)
@@
     (property "Sheetfile" "PCB.kicad_sch")
     (property "Sheetname" "")
-    (property "dnp" "")
     (property "ki_description" "Unpolarized capacitor, small symbol")
     (property "ki_keywords" "capacitor cap")
@@
     (property "Sheetfile" "PCB.kicad_sch")
     (property "Sheetname" "")
-    (property "dnp" "")
-    (property "ki_description" "Low-drop Voltage Regulator, Io up to 500mA, Fixed Vo 5.0V, TO-252 (DPAK)")
-    (property "ki_keywords" "LDO regulator voltage")
+    (property "ki_description" "Positive 1.5A 35V Linear Regulator, Fixed Output 5V, TO-220/TO-263/TO-252")
+    (property "ki_keywords" "Voltage Regulator 1.5A Positive")
     (attr smd)
     (fp_text reference "U6" (at 0 -4.5 90) (layer "F.SilkS")
         (effects (font (size 1 1) (thickness 0.15)))
     )
-    (fp_text value "LF50_TO252" (at 0 4.5 90) (layer "F.Fab")
+    (fp_text value "L7805" (at 0 4.5 90) (layer "F.Fab")
         (effects (font (size 1 1) (thickness 0.15)))
     )
@@
       (stroke (width 0.1) (type solid)) (layer "F.Fab"))
     (pad "1" smd roundrect (at -5.04 -2.28 90) (size 2.2 1.2) (layers "F.Cu" "F.Paste" "F.Mask") (roundrect_rratio 0.208333)
-      (net 43 "Net-(D6-A)") (pinfunction "VI") (pintype "power_in"))
+      (net 43 "Net-(D6-A)") (pinfunction "IN") (pintype "power_in"))
     (pad "2" smd roundrect (at -0.415 -1.525 90) (size 3.05 2.75) (layers "F.Cu" "F.Paste") (roundrect_rratio 0.090909)
       (net 3 "TS-") (pinfunction "GND") (pintype "power_in"))
@@
       (net 3 "TS-") (pinfunction "GND") (pintype "power_in"))
     (pad "3" smd roundrect (at -5.04 2.28 90) (size 2.2 1.2) (layers "F.Cu" "F.Paste" "F.Mask") (roundrect_rratio 0.208333)
-      (net 2 "+5V") (pinfunction "VO") (pintype "power_out"))
+      (net 2 "+5V") (pinfunction "OUT") (pintype "power_out"))
     (model "${KICAD6_3DMODEL_DIR}/Package_TO_SOT_SMD.3dshapes/TO-252-2.wrl"
       (offset (xyz 0 0 0))
@@
       (net 1 "GND") (pinfunction "GNDS") (pintype "power_out"))
   )
+  (footprint "Jumper:SolderJumper-2_P1.3mm_Open_RoundedPad1.0x1.5mm" (layer "F.Cu")
+    (at 134.65 91.2)
+    (descr "SMD Solder Jumper, 1x1.5mm, rounded Pads, 0.3mm gap, open")
+    (tags "solder jumper open")
+    (property "Sheetfile" "PCB.kicad_sch")
+    (property "Sheetname" "")
+    (property "ki_description" "Solder Jumper, 2-pole, open")
+    (property "ki_keywords" "solder jumper SPST")
+    (attr exclude_from_pos_files)
+    (fp_text reference "JP1" (at -2.53 0.07 90) (layer "F.SilkS")
+        (effects (font (size 1 1) (thickness 0.15)))
+    )
+    (fp_text value "SolderJumper_2_Open" (at 0 1.9) (layer "F.Fab")
+        (effects (font (size 1 1) (thickness 0.15)))
+    )
+    (fp_line (start -1.4 0.3) (end -1.4 -0.3)
+      (stroke (width 0.12) (type solid)) (layer "F.SilkS"))
+    (fp_line (start -0.7 -1) (end 0.7 -1)
+      (stroke (width 0.12) (type solid)) (layer "F.SilkS"))
+    (fp_line (start 0.7 1) (end -0.7 1)
+      (stroke (width 0.12) (type solid)) (layer "F.SilkS"))
+    (fp_line (start 1.4 -0.3) (end 1.4 0.3)
+      (stroke (width 0.12) (type solid)) (layer "F.SilkS"))
+    (fp_arc (start -1.4 -0.3) (mid -1.194975 -0.794975) (end -0.7 -1)
+      (stroke (width 0.12) (type solid)) (layer "F.SilkS"))
+    (fp_arc (start -0.7 1) (mid -1.194975 0.794975) (end -1.4 0.3)
+      (stroke (width 0.12) (type solid)) (layer "F.SilkS"))
+    (fp_arc (start 0.7 -1) (mid 1.194975 -0.794975) (end 1.4 -0.3)
+      (stroke (width 0.12) (type solid)) (layer "F.SilkS"))
+    (fp_arc (start 1.4 0.3) (mid 1.194975 0.794975) (end 0.7 1)
+      (stroke (width 0.12) (type solid)) (layer "F.SilkS"))
+    (fp_line (start -1.65 -1.25) (end -1.65 1.25)
+      (stroke (width 0.05) (type solid)) (layer "F.CrtYd"))
+    (fp_line (start -1.65 -1.25) (end 1.65 -1.25)
+      (stroke (width 0.05) (type solid)) (layer "F.CrtYd"))
+    (fp_line (start 1.65 1.25) (end -1.65 1.25)
+      (stroke (width 0.05) (type solid)) (layer "F.CrtYd"))
+    (fp_line (start 1.65 1.25) (end 1.65 -1.25)
+      (stroke (width 0.05) (type solid)) (layer "F.CrtYd"))
+    (pad "1" smd custom (at -0.65 0) (size 1 0.5) (layers "F.Cu" "F.Mask")
+      (net 43 "Net-(D6-A)") (pinfunction "A") (pintype "passive") (zone_connect 2)
+      (options (clearance outline) (anchor rect))
+      (primitives
+        (gr_circle (center 0 0.25) (end 0.5 0.25) (width 0) (fill yes))
+        (gr_circle (center 0 -0.25) (end 0.5 -0.25) (width 0) (fill yes))
+        (gr_poly
+          (pts
+            (xy 0.5 0.75)
+            (xy 0 0.75)
+            (xy 0 -0.75)
+            (xy 0.5 -0.75)
+          )
+          (width 0) (fill yes))
+      ))
+    (pad "2" smd custom (at 0.65 0) (size 1 0.5) (layers "F.Cu" "F.Mask")
+      (net 2 "+5V") (pinfunction "B") (pintype "passive") (zone_connect 2)
+      (options (clearance outline) (anchor rect))
+      (primitives
+        (gr_circle (center 0 0.25) (end 0.5 0.25) (width 0) (fill yes))
+        (gr_circle (center 0 -0.25) (end 0.5 -0.25) (width 0) (fill yes))
+        (gr_poly
+          (pts
+            (xy 0 0.75)
+            (xy -0.5 0.75)
+            (xy -0.5 -0.75)
+            (xy 0 -0.75)
+          )
+          (width 0) (fill yes))
+      ))
+  )
   (footprint "Capacitor_SMD:CP_Elec_6.3x7.7" (layer "F.Cu")
