File: pcb/PCB.kicad_pcb (KiCad board)
At the start: 4 copper layers, 100 x 60 mm, 80 parts, among them J1 TE 770966-2, J2 JST B04B-XASK, J3 Conn_01x02, J4 Conn_01x02, Q1 IRLZ44N, Q2 MMBT3904, Q3 IRLZ44N, U1 TL431D, U2 LMV331, U3 UCC12040DVE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

Commit message: TSSI update 3-29-25 initial
Parts:
- removed D2: LED-Green, LED_SMD:LED_0603_1608Metric
- removed D8, D9: SSB43L, Diode_SMD:D_SMB
- removed Q1: IRLZ44N, IRLZ44NSTRLPBF:NMOSGDS_D2PAK_INF
- removed R10: 2.2k, Resistor_SMD:R_0603_1608Metric
- removed R22: 220k, Resistor_SMD:R_0603_1608Metric
- removed R7: 10k, Resistor_SMD:R_0603_1608Metric
- removed R8: 1k, Resistor_SMD:R_0603_1608Metric
- added C20: 0.1u, Capacitor_SMD:C_0603_1608Metric, F.Cu at (154.0, 134.1)
- added C21: 0.1u, Capacitor_SMD:C_0603_1608Metric, F.Cu at (161.8, 105.8)
- added C22: 1u, Capacitor_SMD:C_0603_1608Metric, F.Cu at (154.0, 137.2)
- added D13: LED-Green, LED_SMD:LED_0603_1608Metric, F.Cu at (152.3, 105.8)
- added D14: LED-Red, LED_SMD:LED_0603_1608Metric, F.Cu at (175.9, 136.8)
- added J6: Conn_01x04, Connector_TE-Connectivity:TE_MATE-N-LOK_1-770968-x_2x02_P4.14mm_Horizontal, F.Cu at (191.7, 128.8)
- added Q4: IRLZ44N, IRLZ44NSTRLPBF:NMOSGDS_D2PAK_INF, F.Cu at (158.3, 112.3)
- added Q5: MMBT3904, Package_TO_SOT_SMD:SOT-23, F.Cu at (170.2, 119.8)
- added Q6: IRLZ44N, IRLZ44NSTRLPBF:NMOSGDS_D2PAK_INF, F.Cu at (176.0, 130.3)
- added R30: 220k, Resistor_SMD:R_0603_1608Metric, F.Cu at (171.1, 110.4)
- added R31: 1k, Resistor_SMD:R_0603_1608Metric, F.Cu at (170.5, 114.8)
- added R32: 22k, Resistor_SMD:R_0603_1608Metric, F.Cu at (174.1, 110.3)
- added R33: 220k, Resistor_SMD:R_0603_1608Metric, F.Cu at (169.9, 117.2)
- added R34: 22k, Resistor_SMD:R_0603_1608Metric, F.Cu at (153.6, 127.8)
- added R35: 2.2k, Resistor_SMD:R_0603_1608Metric, F.Cu at (155.5, 105.8)
- added R36: 22k, Resistor_SMD:R_0603_1608Metric, F.Cu at (161.7, 134.9)
- added R37: 220k, Resistor_SMD:R_0603_1608Metric, F.Cu at (157.0, 139.5)
- added R38: 100k, Resistor_SMD:R_0603_1608Metric, F.Cu at (158.2, 130.2)
- added R39: 1k, Resistor_SMD:R_0603_1608Metric, F.Cu at (158.1, 128.3)
- added R40: 1k, Resistor_SMD:R_0603_1608Metric, F.Cu at (172.4, 136.8)
- added U8: CD4093BM96, Package_SO:SOIC-14_3.9x8.7mm_P1.27mm, F.Cu at (163.4, 122.8)
- added U9: LM555xN, footprints 555:M08A-L, F.Cu at (158.0, 135.0)
- D3: value LED-Red -> LED-Yellow
- R15: value 1k -> 2.2k
- RV1: value 10k -> R_Potentiometer
- moved J4 19.3 mm to (180.3, 94.2)
- moved J2 12.9 mm to (170.7, 143.7)
- moved D3 12.6 mm to (169.1, 79.1)
- moved Q3 12.5 mm to (162.1, 81.4)
- moved R15 12.2 mm to (169.1, 82.8)
- moved H2 11.8 mm to (190.1, 69.3)
- moved H4 11.8 mm to (190.1, 119.3)
- moved H1 11.8 mm to (100.1, 69.3)
- moved H3 11.8 mm to (100.1, 119.3)
- moved C11 11.5 mm to (135.3, 80.8)
- moved C2 11.5 mm to (128.6, 75.3)
- moved J3 11.5 mm to (180.3, 82.9)
- moved R1 11.5 mm to (121.4, 102.0)
- moved R16 11.5 mm to (153.8, 97.2)
- moved R2 11.5 mm to (118.1, 102.0)
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Connections:
- C6 pad 1: +5V@GLV -> +12V
- D3 pad 1: /Ext-LED-RED -> /Ext-LED-AMBER_AFT
- J2 pad 2: +5V@GLV -> unconnected-(J2-Pin_2-Pad2)
- J2 pad 3: /Ext-LED-Green -> /Ext-LED-RED
- J2 pad 4: /Ext-LED-RED -> /Ext-LED-GREEN
- Q3 pad 2: /Ext-LED-RED -> /Ext-LED-AMBER_AFT
- R11 pad 1: +5V@GLV -> +12V
- R15 pad 2: +5V@GLV -> +12V
- R20 pad 1: Net-(D9-K) -> +12V
- R9 pad 2: +5V@GLV -> +12V
- U5 pad 8: +5V@GLV -> +12V
Routing:
- net /Ext-LED-AMBER_AFT: track 0.00 -> 75.4 mm
- net /Ext-LED-GREEN: track 0.00 -> 56.5 mm, vias 0 -> 1
- net Net-(R16-Pad1): track 60.4 -> 14.8 mm, vias 2 -> 0
- net /Ext-LED-RED: track 51.3 -> 14.9 mm
- net +12V: track 23.8 -> 59.6 mm, vias 0 -> 8
- net /Ext-LED-Green: track 30.8 -> 0.00 mm
- net GND: track 44.8 -> 74.6 mm, vias 13 -> 16
- net IMD Fault: track 0.00 -> 29.6 mm, vias 0 -> 1
- net BMS Fault: track 0.00 -> 26.0 mm, vias 0 -> 1
- net Net-(Q5-C): track 0.00 -> 24.7 mm, vias 0 -> 2
- net Net-(U8-J=*A-B): track 0.00 -> 16.5 mm
- net Net-(U9-THR): track 0.00 -> 10.8 mm
- net Net-(Q6-G): track 0.00 -> 9.40 mm
- net Net-(U9-DIS): track 0.00 -> 7.91 mm
- net Net-(D5-A): track 8.53 -> 14.1 mm
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- added copper zone on In1.Cu, net +12V
- added copper zone on B.Cu, net GND
- added copper zone on F.Cu, net GND
- removed copper zone on In1.Cu, net +5V@GLV
Other:
- board size 100 x 60 mm -> 234.5 x 84.8 mm
- board text added: "Bronco Racing TSSI + Voltage Indicator + RTML REV 4"
- board text added: "Light PCB REV 4 2025 R. Kisser N. Banasky"
- board text added: "Reroute all 5glv to a specific conection of it, all 12v are connected"
- board text removed: "+5V"
- board text removed: "Bronco Racing TSAL + Voltage Indicator REV 3"
- board text removed: "TSAL REV 3 2024 J. Iwick J. LeFevre"

Commit message: Kicad 9 preparation
Other:
- board size 234.5 x 84.8 mm -> 100.5 x 82.8 mm
Changed lines of the file:
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@@
 		(layer "F.SilkS")
-	)
-	(gr_line
-		(start 61.135 122.77)
-		(end 61.135 62.77)
-		(stroke
-			(width 0.1)
-			(type default)
-		)
-		(layer "Edge.Cuts")
-	)
-	(gr_line
-		(start 61.135 62.77)
-		(end -38.865 62.77)
-		(stroke
-			(width 0.1)
-			(type default)
-		)
-		(layer "Edge.Cuts")
 	)
 	(gr_rect
@@
 		(layer "Edge.Cuts")
 	)
-	(gr_line
-		(start -38.865 62.77)
-		(end -38.865 122.77)
-		(stroke
-			(width 0.1)
-			(type default)
-		)
-		(layer "Edge.Cuts")
-	)
-	(gr_rect
-		(start -38.865 62.77)
-		(end 61.135 122.77)
-		(stroke
-			(width 0.1)
-			(type default)
-		)
-		(fill no)
-		(layer "Edge.Cuts")
-	)
-	(gr_line
-		(start -38.865 122.77)
-		(end 61.135 122.77)
-		(stroke
-			(width 0.1)
-			(type default)
-		)
-		(layer "Edge.Cuts")
-	)
