File: pcb/PCB.kicad_sch (KiCad schematic)
At the start: 99 parts, among them J1 TE 770966-2, J2 JST B04B-XASK, J3 Conn_01x02, J4 Conn_01x02, J5 TE 770966-2, J6 Conn_01x04, Q2 MMBT3904, Q3 IRLZ44N, Q4 IRLZ44N, Q5 MMBT3904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

Commit message: Kicad 9 preparation
Connections:
- no-connect marks 1 -> 34
Changed lines of the file:
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@@
+	)
+	(no_connect
+		(at 207.01 142.24)
+	)
+	(no_connect
+		(at 363.22 -15.24)
+	)
+	(no_connect
+		(at 373.38 -15.24)
+	)
+	(no_connect
+		(at 391.16 -22.86)
+	)
+	(no_connect
+		(at 391.16 -13.97)
+	)
+	(no_connect
+		(at 391.16 -11.43)
+	)
+	(no_connect
+		(at 391.16 -21.59)
+	)
+	(no_connect
+		(at 369.57 -31.75)
+	)
+	(no_connect
+		(at 375.92 -26.67)
+	)
+	(no_connect
+		(at 375.92 -21.59)
+	)
+	(no_connect
+		(at 391.16 -16.51)
+	)
+	(no_connect
+		(at 369.57 -34.29)
 	)
 	(no_connect
 		(at 464.82 130.81)
 	)
-	(bus_entry
-		(at 0 0)
-		(size 2.54 2.54)
-		(stroke
-			(width 0)
-			(type default)
-		)
+	(no_connect
+		(at 391.16 -8.89)
+	)
+	(no_connect
+		(at 436.88 -3.81)
+	)
+	(no_connect
+		(at 135.89 137.16)
+	)
+	(no_connect
+		(at 207.01 144.78)
+	)
+	(no_connect
+		(at 135.89 139.7)
+	)
+	(no_connect
+		(at 436.88 -21.59)
+	)
+	(no_connect
+		(at 391.16 -6.35)
+	)
+	(no_connect
+		(at 436.88 -19.05)
+	)
+	(no_connect
+		(at 391.16 -3.81)
+	)
+	(no_connect
+		(at 360.68 -26.67)
+	)
+	(no_connect
+		(at 207.01 137.16)
+	)
+	(no_connect
+		(at 207.01 134.62)
+	)
+	(no_connect
+		(at 436.88 -16.51)
+	)
+	(no_connect
+		(at 207.01 138.43)
+	)
+	(no_connect
+		(at 135.89 142.24)
+	)
+	(no_connect
+		(at 391.16 -19.05)
+	)
+	(no_connect
+		(at 381 -15.24)
+	)
+	(no_connect
+		(at 360.68 -21.59)
+	)
+	(no_connect
+		(at 207.01 139.7)
+	)
+	(no_connect
+		(at 207.01 132.08)
+	)
+	(no_connect
+		(at 436.88 -13.97)
 	)
 	(wire

Commit message: For gerbers
Parts:
- removed C16, C17: 500V 3.9u, Capacitor_SMD:C_Elec_10x10.2, symbol Device:C_Small
- removed J5: TE 770966-2, Connector_TE-Connectivity:TE_MATE-N-LOK_1-770966-x_1x02_P4.14mm_Horizontal, symbol Connector_Generic:Conn_01x02
- removed L3: 1m, Inductor_SMD:L_1210_3225Metric, symbol Device:L
- removed TP7: TestPoint, TestPoint:TestPoint_Keystone_5019_Minature, symbol Connector:TestPoint
- removed U10: UCC12040DVE, footprints:SO_0DVER_TEX, symbol 2023-11-19_21-51-37:UCC12040DVE
Connections:
- no-connect marks 34 -> 10
